File: Dash 6.8_V0.1/Dash 6.8.kicad_pcb (KiCad board)
At the start: 2 copper layers, 156 x 66 mm, 140 parts, among them J1 USB_B_Mini, J2 Conn_01x04, J3 5-1814400-1, J4 Conn_01x40_MountingPin, J5 776262-1, Q1 DMP3013SFV-7, SW1 SW_Push, U1 REF3333, U11 ILD207T, U12 MCP6001-OT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

Commit message: исправление платы V01
Parts:
- added R25: 10k, Resistor_SMD:R_0603_1608Metric, F.Cu at (178.8, 89.2)
- J3: value 5-1814400-1 -> 20279-001E-03
- moved C5 0.60 mm to (181.4, 89.8)
- moved C23 0.55 mm to (181.4, 88.2)
Connections:
- U4 pad 171: unconnected-(U4-PDR_ON-Pad171) -> Net-(U4-PDR_ON)
- U4 pad 48: unconnected-(U4-BYPASS_REG-Pad48) -> GND
Routing:
- net Net-(U4-PDR_ON): track 0.00 -> 10.4 mm
- net +3.3V: track 591.6 -> 592.3 mm
- net GND: vias 277 -> 276
