File: Dash 6.8_V0.1/Dash 6.8.kicad_sch (KiCad schematic)
At the start: 140 parts, among them J1 USB_B_Mini, J2 Conn_01x04, J3 20279-001E-03, J4 Conn_01x40_MountingPin, J5 776262-1, Q1 DMP3013SFV-7, SW1 SW_Push, U1 REF3333, U11 ILD207T, U12 MCP6001-OT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

Commit message: исправление платы V01
Parts:
- added R25: 10k, Resistor_SMD:R_0603_1608Metric, symbol Device:R
Connections:
- net +3.3V: now also R25.2
- net GND: now also U4.48 (BYPASS_REG)
- net at U4.171 (PDR_ON): now also R25.1
- no-connect marks 80 -> 78
Other:
- moved on the sheet: 12v1, 5v1, C1, C10, C11, C12, C13, C14, C15, C16, C17, C18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
