File: Dash 6.8_V0.2/Dash 6.8.kicad_sch (KiCad schematic)
At the start: 151 parts, among them J1 USB_B_Mini, J2 Conn_01x04, J3 20279-001E-03, J4 Conn_01x40_MountingPin, J5 776262-1, J6 Conn_01x04, Q1 DMP3013SFV-7, SW1 SW_Push, SW2 SW_Push, U1 REF3333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

Commit message: исправление платы V02
Parts:
- added R38: 10k, Resistor_SMD:R_0603_1608Metric, symbol Device:R
Connections:
- net +3.3V: now also R38.2
- net GND: now also R31.2, U12.1, U12.4 (-), U4.48 (BYPASS_REG)
- net at U4.171 (PDR_ON): now also R38.1
- no-connect marks 109 -> 107
Other:
- moved on the sheet: 12v1, 5v1, C1, C10, C11, C12, C13, C14, C15, C16, C17, C18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
